File: hardware/relay_channel.kicad_sch (KiCad schematic)
At the start: 9 parts, among them K1 TQ2-L2-5V, Q1 MMBT2222A, Q2 MMBT2222A

Commit message: Rev0: named analog nets, both relay poles, HV netclass, smaller board
Restore the HV netclass (the real bug)
--------------------------------------
nanovolt-divider.kicad_dru conditions all three 450 V rules on NetClass == 'HV',
but the project file had "netclass_patterns": [] and no HV class, so every one of
them matched nothing. DRC reported "0 violations" whether the board was safe or
not. The original patterns matched auto-generated names like Net-(J3-Pin_1) and
were dropped when KiCad rewrote the project file.

The class is back with the patterns spelled out - /HV_IN_P and /HV_DIV, never a
"HV*" wildcard, which would sweep in HV_SENSE (a 3.3 V logic line). Verified by
moving R34 next to K5 on a scratch copy and confirming the rules fire; restoring
them immediately exposed 25 real clearance/creepage violations in the old
placement, now fixed.

gen_schematics.py no longer overwrites .kicad_pro (write_once): it emits a
25-line stub, and KiCad owns the 702-line file that holds the netclass.

Schematic
---------
* Analog nets carry real labels instead of /POLARITY (K4)/A_COM and
  Net-(J4-Pin_1): SRC_P, SRC_RTN, NORMAL_IN_P/N, RANGE_BUS, R*_IN, R*_OUT,
  INJ_NODE, MEAS_NODE, ANALOG_RTN, HV_IN_P, HV_DIV. This is also what gives the
  HV netclass stable patterns to match.
* K1..K3 use both poles: SRC_P -> A_COM -> A_NO -> R -> B_NO -> B_COM ->
  RANGE_BUS, so a deselected high leg is isolated at both ends.
* Control ground is DGND, not the global GND, so it cannot merge with the
  floating analog return.
* J7/J8/J9 use project symbols with the module's own pin names (SCL_IO22, IO35)
  instead of Conn_01x04 Pin_1..Pin_4. Pin geometry is unchanged, so no wire moved.
* Removed from the board: J4 (HV IN- is a panel-to-panel wire to SW1 lug 6), R26
  and SW1 lug 7 (R25's 100k already holds HV_SENSE low off the HV throw). Added
  C5 10 nF to stiffen the 100k against pickup on the IO35 harness. The two
  off-board lugs are documented in a panel-wiring note on the root sheet.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
Connections:
- net GND renamed DGND
Changed lines of the file:
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@@
 	(wire (pts (xy 48.26 63.5) (xy 48.26 67.31)) (stroke (width 0) (type default)))
 	(wire (pts (xy 48.26 74.93) (xy 48.26 77.47)) (stroke (width 0) (type default)))
-	(symbol (lib_id "power:GND") (at 48.26 77.47 0) (unit 1) (body_style 1) (exclude_from_sim no) (in_bom yes) (on_board yes) (in_pos_files yes) (dnp no)
+	(symbol (lib_id "nanovolt-divider:DGND") (at 48.26 77.47 0) (unit 1) (body_style 1) (exclude_from_sim no) (in_bom yes) (on_board yes) (in_pos_files yes) (dnp no)
 	  (property "Reference" "#PWR101" (at 48.26 83.82 0) (hide yes) (show_name no) (do_not_autoplace no) (effects (font (size 1.27 1.27)) (justify left)))
-	  (property "Value" "GND" (at 48.26 81.28 0) (show_name no) (do_not_autoplace no) (effects (font (size 1.27 1.27)) (justify left)))
+	  (property "Value" "DGND" (at 48.26 81.28 0) (show_name no) (do_not_autoplace no) (effects (font (size 1.27 1.27)) (justify left)))
 	  (property "Footprint" "" (at 48.26 77.47 0) (hide yes) (show_name no) (do_not_autoplace no) (effects (font (size 1.27 1.27)) (justify left)))
 	  (property "Datasheet" "" (at 48.26 77.47 0) (hide yes) (show_name no) (do_not_autoplace no) (effects (font (size 1.27 1.27)) (justify left)))
-	  (property "Description" "Power symbol creates a global label with name \\\"GND\\\" , ground" (at 48.26 77.47 0) (hide yes) (show_name no) (do_not_autoplace no) (effects (font (size 1.27 1.27)) (justify left)))
+	  (property "Description" "Control-section digital ground (MCP23017, TMP117, relay coil drivers, ESP32 harness). Never tied to the floating analog return." (at 48.26 77.47 0) (hide yes) (show_name no) (do_not_autoplace no) (effects (font (size 1.27 1.27)) (justify left)))
 	  (pin "1")
 	  (instances (project "nanovolt-divider"
@@
 	(wire (pts (xy 48.26 127) (xy 48.26 130.81)) (stroke (width 0) (type default)))
 	(wire (pts (xy 48.26 138.43) (xy 48.26 140.97)) (stroke (width 0) (type default)))
-	(symbol (lib_id "power:GND") (at 48.26 140.97 0) (unit 1) (body_style 1) (exclude_from_sim no) (in_bom yes) (on_board yes) (in_pos_files yes) (dnp no)
+	(symbol (lib_id "nanovolt-divider:DGND") (at 48.26 140.97 0) (unit 1) (body_style 1) (exclude_from_sim no) (in_bom yes) (on_board yes) (in_pos_files yes) (dnp no)
 	  (property "Reference" "#PWR103" (at 48.26 147.32 0) (hide yes) (show_name no) (do_not_autoplace no) (effects (font (size 1.27 1.27)) (justify left)))
-	  (property "Value" "GND" (at 48.26 144.78 0) (show_name no) (do_not_autoplace no) (effects (font (size 1.27 1.27)) (justify left)))
+	  (property "Value" "DGND" (at 48.26 144.78 0) (show_name no) (do_not_autoplace no) (effects (font (size 1.27 1.27)) (justify left)))
 	  (property "Footprint" "" (at 48.26 140.97 0) (hide yes) (show_name no) (do_not_autoplace no) (effects (font (size 1.27 1.27)) (justify left)))
 	  (property "Datasheet" "" (at 48.26 140.97 0) (hide yes) (show_name no) (do_not_autoplace no) (effects (font (size 1.27 1.27)) (justify left)))
-	  (property "Description" "Power symbol creates a global label with name \\\"GND\\\" , ground" (at 48.26 140.97 0) (hide yes) (show_name no) (do_not_autoplace no) (effects (font (size 1.27 1.27)) (justify left)))
+	  (property "Description" "Control-section digital ground (MCP23017, TMP117, relay coil drivers, ESP32 harness). Never tied to the floating analog return." (at 48.26 140.97 0) (hide yes) (show_name no) (do_not_autoplace no) (effects (font (size 1.27 1.27)) (justify left)))
 	  (pin "1")
 	  (instances (project "nanovolt-divider"
