File: hardware/control.kicad_sch (KiCad schematic)
At the start: 11 parts, among them J7 ESP32_DISP_P1, J8 ESP32_DISP_CN1, U1 MCP23017-E/SO, U2 TMP275AIDR

Commit message: Wire the harness to the display module in hand; add the enclosure
The Rev A pads were drawn for an assumed ESP32-2432S028R pinout (P1 =
TX/RX/VIN/GND, CN1 = GND/IO22/IO27/3V3). The Cheap Yellow Display in hand
has UART/power (RXD, TXD, GND, 5V), 3V3 (3.3V, IO35, nc, GND) and SPI
(IO23, IO19, IO18, IO27) connectors, and no IO22.

The board is fabricated, so only the harness and the firmware pins move:
I2C is now SDA = IO27, SCL = IO18, and J8 is fed by two pigtails. J7's
silk numbers are reversed against the module (module pin 3 is GND, pad 3
is +5V), so the docs say to land wires by signal name.

The netlist is unchanged. The symbols' pin names and descriptions follow
the module. The harness footprints are frozen as fabricated
(HARNESS_PADS_REV_A), so the library still matches the board. DRC parity
gains 2 footprint_symbol_field_mismatch warnings (J7/J8 Description),
because the board's copy was deliberately left as fabricated.

Also adds the SOLIDWORKS enclosure parts with their 3MF/3DXML exports,
marks those formats binary, and ignores SOLIDWORKS lock files.

Co-Authored-By: Claude Opus 5.5 <noreply@anthropic.com>
Other:
- note added: "ESP32 2.8in touch display module (Cheap Yellow Display, ESP32-2432S028R type) - off-board, 3 pigtails: UART: RXD / TXD / GND / 5V -> J7: 5V -> pad 3, GND -> pad 4 (reversed!). USB 5V, powers the relay coils. 3V3 : 3.3V / IO35 / nc / GND -> J8: GND -> pad 1, 3.3V -> pad 4. Module LDO feeds U1, U2, pull-ups. SPI : IO23 / IO19 / IO18 / IO27 -> J8: IO18 (SCL) -> pad 2, IO27 (SDA) -> pad 3. IO18 share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"
- note removed: "ESP32 2.8in touch display module (ESP32-2432S028R type, ELEGOO) - off-board, connected by 3 harnesses: P1 : TX / RX / VIN(5V) / GND -> VIN is the module's USB 5 V rail; it powers the relay coils (+5V). CN1: GND / IO22 / IO27 / 3V3 -> I2C: SCL = IO22, SDA = IO27. 3V3 from the module LDO feeds U1, U2, pull-ups. I2C addresses: MCP23017 0x20 (A2:A0 = 000), TMP275 0x48 (A2:A0 = GND). 4.7k pull-ups to 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"
- moved on the sheet: J7
Changed lines of the file:
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@@
 	  (property "Footprint" "nanovolt-divider:J_ESP32_P1_WirePads" (at 38.1 45.72 0) (hide yes) (show_name no) (do_not_autoplace no) (effects (font (size 1.27 1.27)) (justify left)))
 	  (property "Datasheet" "~" (at 38.1 45.72 0) (hide yes) (show_name no) (do_not_autoplace no) (effects (font (size 1.27 1.27)) (justify left)))
-	  (property "Description" "Soldered pigtail to ESP32-2432S028R (ELEGOO 2.8in) connector P1: 3 VIN(5V), 4 GND. TX(IO1) pin 1 and RX(IO3) pin 2 are cut back at the cable." (at 38.1 45.72 0) (hide yes) (show_name no) (do_not_autoplace no) (effects (font (size 1.27 1.27)) (justify left)))
+	  (property "Description" "Soldered pigtail from the display module UART/power connector (RXD, TXD, GND, 5V): pad 3 = 5V wire, pad 4 = GND wire (reverse of the module pin order). RXD/TXD cut back at the cable." (at 38.1 45.72 0) (hide yes) (show_name no) (do_not_autoplace no) (effects (font (size 1.27 1.27)) (justify left)))
 	  (pin "3")
 	  (pin "4")
@@
 	  (property "Footprint" "nanovolt-divider:J_ESP32_CN1_WirePads" (at 38.1 76.2 0) (hide yes) (show_name no) (do_not_autoplace no) (effects (font (size 1.27 1.27)) (justify left)))
 	  (property "Datasheet" "~" (at 38.1 76.2 0) (hide yes) (show_name no) (do_not_autoplace no) (effects (font (size 1.27 1.27)) (justify left)))
-	  (property "Description" "Soldered pigtail to ESP32-2432S028R connector CN1: 1 GND, 2 IO22 (SCL), 3 IO27 (SDA), 4 3V3" (at 38.1 76.2 0) (hide yes) (show_name no) (do_not_autoplace no) (effects (font (size 1.27 1.27)) (justify left)))
+	  (property "Description" "Two display-module pigtails: 1 GND and 4 3.3V from the 3V3 connector (3.3V, IO35, nc, GND); 2 IO18 (SCL) and 3 IO27 (SDA) from the SPI connector (IO23, IO19, IO18, IO27)." (at 38.1 76.2 0) (hide yes) (show_name no) (do_not_autoplace no) (effects (font (size 1.27 1.27)) (justify left)))
 	  (pin "1")
 	  (pin "2")
@@
 	  ))
 	)
-	(text "ESP32 2.8in touch display module (ESP32-2432S028R type, ELEGOO) - off-board, connected by 3 harnesses:\n  P1 : TX / RX / VIN(5V) / GND   -> VIN is the module's USB 5 V rail; it powers the relay coils (+5V).\n  CN1: GND / IO22 / IO27 / 3V3    -> I2C: SCL = IO22, SDA = IO27. 3V3 from the module LDO feeds U1, U2, pull-ups.\nI2C addresses: MCP23017 0x20 (A2:A0 = 000), TMP275 0x48 (A2:A0 = GND). 4.7k pull-ups to 3V3 on this board.\nMCP23017 GPB0..GPB7 -> K4 S/R, K1 S/R, K2 S/R, K3 S/R; GPA0 -> K5 RESET, GPA1 -> K5 SET (layout order).\nMCP23017 GPA2..GPA7 are spare; the ESP32 side has no board connection beyond P1 and CN1." (at 172.72 143.51 0) (effects (font (size 1.0 1.0)) (justify left bottom)))
+	(text "ESP32 2.8in touch display module (Cheap Yellow Display, ESP32-2432S028R type) - off-board, 3 pigtails:\n  UART: RXD / TXD / GND / 5V       -> J7: 5V -> pad 3, GND -> pad 4 (reversed!). USB 5V, powers the relay coils.\n  3V3 : 3.3V / IO35 / nc / GND     -> J8: GND -> pad 1, 3.3V -> pad 4. Module LDO feeds U1, U2, pull-ups.\n  SPI : IO23 / IO19 / IO18 / IO27  -> J8: IO18 (SCL) -> pad 2, IO27 (SDA) -> pad 3. IO18 shared w/ SD slot.\nRev A pad silk (P1 3/4, CN1 1-4) follows an assumed pinout: land wires by signal name, not by number.\nI2C addresses: MCP23017 0x20 (A2:A0 = 000), TMP275 0x48 (A2:A0 = GND). 4.7k pull-ups to 3V3 on this board.\nMCP23017 GPB0..GPB7 -> K4 S/R, K1 S/R, K2 S/R, K3 S/R; GPA0 -> K5 RESET, GPA1 -> K5 SET (layout order).\nMCP23017 GPA2..GPA7 are spare; the ESP32 side has no board connection beyond J7 and J8." (at 172.72 143.51 0) (effects (font (size 1.0 1.0)) (justify left bottom)))
 	(text "ESP32 display module harness" (at 25.4 30.48 0) (effects (font (size 2.0 2.0)) (justify left bottom)))
 	(text "MCP23017 -> relay coil drivers" (at 66.04 80.01 0) (effects (font (size 2.0 2.0)) (justify left bottom)))
